File: ntg393/ntg393.kicad_sch (KiCad schematic)
At the start: 47 parts, among them J1 AudioJack, J2 Speaker, J3 UART1, J4 Pot, J5 Joystick, J6 GND, J7 DACOUT, SW1 UP, SW2 LEFT, SW3 DOWN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

Commit message: updating files
Connections:
- net PA8 is gone; now on net PA24: J3.2 (B), U2.J1_4 (PA8), U5.1 (1B)
Changed lines of the file:
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@@
+    (stroke (width 0) (type default))
+  )
+  (wire (pts (xy 213.36 31.75) (xy 223.52 31.75))
     (stroke (width 0) (type default))
   )
@@
   )
   (wire (pts (xy 127 165.1) (xy 127 166.37))
+    (stroke (width 0) (type default))
+  )
+  (wire (pts (xy 213.36 39.37) (xy 223.52 39.37))
     (stroke (width 0) (type default))
   )
@@
     )
   )
+  (global_label "PA24" (shape input) (at 223.52 39.37 0) (fields_autoplaced)
+    (effects (font (size 1.27 1.27)) (justify left))
+    (property "Intersheetrefs" "${INTERSHEET_REFS}" (at 231.2828 39.37 0)
+      (effects (font (size 1.27 1.27)) (justify left) hide)
+    )
+  )
   (global_label "PA13" (shape input) (at 82.55 45.72 180) (fields_autoplaced)
     (effects (font (size 1.27 1.27)) (justify right))
@@
     )
   )
+  (global_label "PA24" (shape input) (at 213.36 31.75 180) (fields_autoplaced)
+    (effects (font (size 1.27 1.27)) (justify right))
+    (property "Intersheetrefs" "${INTERSHEET_REFS}" (at 205.5972 31.75 0)
+      (effects (font (size 1.27 1.27)) (justify right) hide)
+    )
+  )
   (global_label "PB24" (shape input) (at 59.69 148.59 180) (fields_autoplaced)
     (effects (font (size 1.27 1.27)) (justify right))
@@
     )
   )
+  (global_label "PA8" (shape input) (at 213.36 39.37 180) (fields_autoplaced)
+    (effects (font (size 1.27 1.27)) (justify right))
+    (property "Intersheetrefs" "${INTERSHEET_REFS}" (at 206.8067 39.37 0)
+      (effects (font (size 1.27 1.27)) (justify right) hide)
+    )
+  )
   (global_label "PB17" (shape input) (at 34.29 119.38 180) (fields_autoplaced)
     (effects (font (size 1.27 1.27)) (justify right))
@@
     )
   )
+  (global_label "PA8" (shape input) (at 223.52 31.75 0) (fields_autoplaced)
+    (effects (font (size 1.27 1.27)) (justify left))
+    (property "Intersheetrefs" "${INTERSHEET_REFS}" (at 230.0733 31.75 0)
+      (effects (font (size 1.27 1.27)) (justify left) hide)
+    )
+  )
